File: Dad_OrganShutters.sch (EAGLE design)
At the start: 3 parts

Commit message: updates
Parts:
- removed R2: (no value), pot:TRIM_US-3223G
Connections:
- net +5V: no longer R2.A
- net GND: no longer R2.E
Other:
- note added: "12 VDC from Syndyne (tip+)"
- note added: "24VDC motor"
- note added: "Cable wire colors RED: +5 BLK: Gnd WHT: 40, Position fdbk ORA: 71, Motor- BLU: 72, Motor+ GRN: N/C SHLD: Gnd at controller"
- note added: "IN1 MOTOR DIR A"
- note added: "IN2 MOTOR DIR B"
- note added: "MOTOR ENABLE"
- note added: "MOTOR+, Blue, 72"
- note added: "MOTOR-, Orange, 71"
- note added: "Motor driver module"
- note added: "Note 73 (Not used)"
- note added: "S1"
- note added: "S2"
- note added: "S3"
- note added: "S4"
- note added: "S5"
- note added: "S6"
- note added: "S7"
- note added: "Shutter position pot"
- note added: "WHT (tag 40)"
- note removed: "12 VDC from Syndyne"
- note removed: "24VDC motor, room 1"
- note removed: "24VDC motor, room 2"
- note removed: "MOTOR1 +"
- note removed: "MOTOR1 -"
- note removed: "MOTOR1_DIRA"
- note removed: "MOTOR1_DIRB"
- note removed: "MOTOR1_ENABLE"
- note removed: "MOTOR2 +"
- note removed: "MOTOR2 -"
- note removed: "MOTOR2_DIRA"
- note removed: "MOTOR2_DIRB"
- note removed: "MOTOR2_ENABLE"
- note removed: "Motor driver module (for 2 DC motors)"
- note removed: "Shutter position pot (each room)"

Commit message: update schematic
Parts:
- added R2, R3, R4, R5, R6, R7, R8: (no value), resistor:R-US_0204/2V
Other:
- note added: "Convert from 12V "levels" from Syndyne to open collector"
- note added: "S1 LSB"
- note added: "S7 MSB"
- note removed: "Note 73 (Not used)"
- note removed: "S1"
- note removed: "S7"
Changed lines of the file:
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@@
 <layer number="97" name="Info" color="7" fill="1" visible="yes" active="yes"/>
 <layer number="98" name="Guide" color="6" fill="1" visible="yes" active="yes"/>
+<layer number="99" name="SpiceOrder" color="5" fill="1" visible="yes" active="yes"/>
 <layer number="100" name="Muster" color="7" fill="1" visible="no" active="no"/>
 <layer number="101" name="Patch_Top" color="12" fill="4" visible="yes" active="yes"/>
@@
 <part name="P+1" library="supply1" deviceset="+5V" device="" value="+5V (tag 32)"/>
 <part name="P+2" library="supply1" deviceset="+5V" device="" value="+5V  (tag 32)"/>
+<part name="R2" library="resistor" deviceset="R-US_" device="0204/2V"/>
+<part name="R3" library="resistor" deviceset="R-US_" device="0204/2V"/>
+<part name="R4" library="resistor" deviceset="R-US_" device="0204/2V"/>
+<part name="R5" library="resistor" deviceset="R-US_" device="0204/2V"/>
+<part name="R6" library="resistor" deviceset="R-US_" device="0204/2V"/>
+<part name="R7" library="resistor" deviceset="R-US_" device="0204/2V"/>
+<part name="R8" library="resistor" deviceset="R-US_" device="0204/2V"/>
 </parts>
 <sheets>
@@
 <wire x1="43.18" y1="185.42" x2="43.18" y2="177.8" width="0.1524" layer="94"/>
 <wire x1="43.18" y1="177.8" x2="17.78" y2="177.8" width="0.1524" layer="94"/>
-<text x="7.62" y="152.4" size="1.778" layer="94" rot="R90">To Syndyne pipe driver board</text>
+<text x="-27.94" y="165.1" size="1.778" layer="94" rot="R90">To Syndyne pipe driver board</text>
 <wire x1="93.98" y1="218.44" x2="106.68" y2="218.44" width="0.1524" layer="94"/>
 <text x="93.98" y="223.52" size="1.778" layer="94">12 VDC from Syndyne (tip+)</text>
@@
 <wire x1="50.8" y1="185.42" x2="50.8" y2="170.18" width="0.1524" layer="94"/>
 <wire x1="50.8" y1="170.18" x2="17.78" y2="170.18" width="0.1524" layer="94"/>
-<wire x1="53.34" y1="185.42" x2="53.34" y2="167.64" width="0.1524" layer="94"/>
-<wire x1="53.34" y1="167.64" x2="17.78" y2="167.64" width="0.1524" layer="94"/>
-<text x="0" y="185.42" size="1.778" layer="94">Note 73 (Not used)</text>
-<text x="12.7" y="182.88" size="1.778" layer="94">S1</text>
-<text x="12.7" y="180.34" size="1.778" layer="94">S2</text>
-<text x="12.7" y="177.8" size="1.778" layer="94">S3</text>
-<text x="12.7" y="175.26" size="1.778" layer="94">S4</text>
-<text x="12.7" y="172.72" size="1.778" layer="94">S5</text>
-<text x="12.7" y="170.18" size="1.778" layer="94">S6</text>
-<text x="12.7" y="167.64" size="1.778" layer="94">S7</text>
+<text x="-25.4" y="185.42" size="1.778" layer="94">S1 LSB</text>
+<text x="-25.4" y="182.88" size="1.778" layer="94">S2</text>
+<text x="-25.4" y="180.34" size="1.778" layer="94">S3</text>
+<text x="-25.4" y="177.8" size="1.778" layer="94">S4</text>
+<text x="-25.4" y="175.26" size="1.778" layer="94">S5</text>
+<text x="-25.4" y="172.72" size="1.778" layer="94">S6</text>
+<text x="-25.4" y="170.18" size="1.778" layer="94">S7 MSB</text>
 <wire x1="66.04" y1="152.4" x2="66.04" y2="185.42" width="0.1524" layer="94"/>
 <text x="66.04" y="152.4" size="1.778" layer="94" rot="R90">MOTOR ENABLE</text>
@@
 SHLD:  Gnd at controller</text>
 <text x="50.8" y="238.76" size="1.778" layer="94">WHT (tag 40)</text>
+<wire x1="-22.86" y1="185.42" x2="-12.7" y2="185.42" width="0.1524" layer="94"/>
+<wire x1="-22.86" y1="182.88" x2="-12.7" y2="182.88" width="0.1524" layer="94"/>
+<wire x1="-22.86" y1="180.34" x2="-10.16" y2="180.34" width="0.1524" layer="94"/>
+<wire x1="-22.86" y1="177.8" x2="-10.16" y2="177.8" width="0.1524" layer="94"/>
+<wire x1="-22.86" y1="175.26" x2="-10.16" y2="175.26" width="0.1524" layer="94"/>
+<wire x1="-22.86" y1="172.72" x2="-12.7" y2="172.72" width="0.1524" layer="94"/>
+<wire x1="-22.86" y1="170.18" x2="-12.7" y2="170.18" width="0.1524" layer="94"/>
+<wire x1="17.78" y1="165.1" x2="76.2" y2="165.1" width="0.1524" layer="94"/>
+<wire x1="76.2" y1="165.1" x2="76.2" y2="185.42" width="0.1524" layer="94"/>
+<text x="-25.4" y="157.48" size="1.778" layer="94">Convert from 12V "levels" from Syndyne to open collector</text>
 </plain>
+<moduleinsts>
+<moduleinst name="ULN2003A" module="MOTORCONTROLLER" x="7.62" y="177.8" rot="R90"/>
+</moduleinsts>
 <instances>
 <instance part="PCB1" gate="G$1" x="60.96" y="205.74" rot="R180"/>
@@
 <instance part="P+1" gate="1" x="73.66" y="261.62"/>
 <instance part="P+2" gate="1" x="114.3" y="154.94"/>
+<instance part="R2" gate="G$1" x="-7.62" y="185.42"/>
+<instance part="R3" gate="G$1" x="-7.62" y="182.88"/>
+<instance part="R4" gate="G$1" x="-7.62" y="180.34"/>
+<instance part="R5" gate="G$1" x="-7.62" y="177.8"/>
+<instance part="R6" gate="G$1" x="-7.62" y="175.26"/>
+<instance part="R7" gate="G$1" x="-7.62" y="172.72"/>
+<instance part="R8" gate="G$1" x="-7.62" y="170.18"/>
 </instances>
 <busses>

Commit message: updated schematic
Parts:
- added R9: (no value), resistor:R-US_0204/2V
Connections:
- net GND: now also R9.1
Other:
- note added: "ENABLE A"
- note added: "ENABLE B"
- note added: "IN1"
- note added: "IN2"
- note added: "IN3"
- note added: "IN4"
- note added: "Last modified July 16, 2017"
- note added: "MOTOR+, Blue 72"
- note added: "MOTOR-, Orange 71"
- note added: "Motor 1"
- note added: "Motor 2"
- note added: "NC"
- note added: "S1-S7 all have pulldowns"
- note removed: "IN1 MOTOR DIR A"
- note removed: "IN2 MOTOR DIR B"
- note removed: "MOTOR ENABLE"
- moved on the sheet: R2, R3, R4, R5, R6, R7, R8
